File: carte ext/carte ext.kicad_pcb (KiCad board)
At the start: 2 copper layers, 86.7 x 56.6 mm, 157 parts, among them J1 Conn_01x02, J10 Conn_01x04, J11 Conn_01x04, J12 Conn_01x04, J13 Conn_01x04, J14 Conn_01x04, J15 Conn_01x04, J16 Conn_01x04, J17 Conn_01x04, J18 Conn_01x04, J19 Conn_01x04, J2 Conn_01x02, J20 Conn_01x04, J21 Conn_02x04_Odd_Even, J22 Conn_02x04_Odd_Even, J23 Conn_02x04_Odd_Even, J24 Conn_02x04_Odd_Even, J25 Conn_02x04_Odd_Even, J26 Conn_02x04_Odd_Even, J27 Conn_02x04_Odd_Even, J28 Conn_02x04_Odd_Even, J29 Conn_02x04_Odd_Even, J3 Conn_01x04, J30 Conn_02x04_Odd_Even, J31 Conn_02x04_Odd_Even, J32 Conn_02x04_Odd_Even, J33 Conn_01x02, J4 Conn_01x04, J5 Conn_01x04, J6 Conn_01x04, J7 Conn_01x04, J8 Conn_01x04, J9 Conn_01x04, U1 PCA9685PW, U2 PCA9685PW, U3 PCA9685PW, U4 PCF8574AT, U5 PCF8574AT

Commit message: on avance bien
Routing:
- net GND: track 459.9 -> 573.6 mm
Changed lines of the file:
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@@
 			(pinfunction "Pin_1")
 			(pintype "passive")
+			(thermal_bridge_angle 45)
 		)
 		(pad "2" thru_hole circle
@@
 		(layer "Edge.Cuts")
 	)
+	(dimension
+		(type orthogonal)
+		(layer "Dwgs.User")
+		(pts
+			(xy 179.05 85.8) (xy 92.4 85.2)
+		)
+		(height 37.75)
+		(orientation 0)
+		(format
+			(prefix "")
+			(suffix "")
+			(units 3)
+			(units_format 0)
+			(precision 4)
+			(suppress_zeroes yes)
+		)
+		(style
+			(thickness 0.1)
+			(arrow_length 1.27)
+			(text_position_mode 0)
+			(arrow_direction outward)
+			(extension_height 0.58642)
+			(extension_offset 0.5)
+			(keep_text_aligned yes)
+		)
+		(gr_text "86,65"
+			(at 135.725 122.4 0)
+			(layer "Dwgs.User")
+			(effects
+				(font
+					(size 1 1)
+					(thickness 0.15)
+				)
+			)
+		)
+	)
+	(dimension
+		(type orthogonal)
+		(layer "Dwgs.User")
+		(pts
+			(xy 135.6 56.4) (xy 135.6 113)
+		)
+		(height -64.3)
+		(orientation 1)
+		(format
+			(prefix "")
+			(suffix "")
+			(units 3)
+			(units_format 0)
+			(precision 4)
+			(suppress_zeroes yes)
+		)
+		(style
+			(thickness 0.1)
+			(arrow_length 1.27)
+			(text_position_mode 0)
+			(arrow_direction outward)
+			(extension_height 0.58642)
+			(extension_offset 0.5)
+			(keep_text_aligned yes)
+		)
+		(gr_text "56,6"
+			(at 70.15 84.7 90)
+			(layer "Dwgs.User")
+			(effects
+				(font
+					(size 1 1)
+					(thickness 0.15)
+				)
+			)
+		)
+	)
 	(segment
 		(start 159.299 82.099)
@@
 		(start 177.239 61.499)
 		(end 177.239 102.719)
-		(width 1.5)
+		(width 2)
 		(layer "F.Cu")
 		(net 1)
@@
 		(start 94.2 102.72)
 		(end 94.2 61.5)
-		(width 1.5)
+		(width 2)
 		(layer "F.Cu")
 		(net 1)
@@
 	)
 	(segment
+		(start 94.21 102.284999)
+		(end 94.21 106.81)
+		(width 2)
+		(layer "B.Cu")
+		(net 1)
+	)
+	(segment
+		(start 134.573959 106.826041)
+		(end 135.7 105.7)
+		(width 2)
+		(layer "B.Cu")
+		(net 1)
+	)
+	(segment
+		(start 103.6 109)
+		(end 104.4 108.2)
+		(width 2)
+		(layer "B.Cu")
+		(net 1)
+	)
+	(segment
 		(start 106.24 70.92)
 		(end 108.79 68.37)
@@
 	)
 	(segment
+		(start 110.371 102.229)
+		(end 122.852959 102.229)
+		(width 2)
+		(layer "B.Cu")
+		(net 1)
+	)
+	(segment
 		(start 132.15 93.8)
 		(end 132.15 103.2)
@@
 	)
 	(segment
+		(start 127.45 106.826041)
+		(end 134.573959 106.826041)
+		(width 2)
+		(layer "B.Cu")
+		(net 1)
+	)
+	(segment
 		(start 176.64108 82.099)
 		(end 167.849 82.099)
@@
 	)
 	(segment
+		(start 122.852959 102.229)
+		(end 127.45 106.826041)
+		(width 2)
+		(layer "B.Cu")
+		(net 1)
+	)
+	(segment
 		(start 142.6 68.294998)
 		(end 140.1 68.294998)
@@
 	)
 	(segment
+		(start 104.4 104.37979)
+		(end 110.45979 98.32)
+		(width 2)
+		(layer "B.Cu")
+		(net 1)
+	)
+	(segment
 		(start 94.2 69.12)
 		(end 94.2 70.322081)
@@
 	)
 	(segment
+		(start 94.21 61.495)
+		(end 94.21 102.284999)
+		(width 2)
+		(layer "B.Cu")
+		(net 1)
+	)
+	(segment
 		(start 117.7 68.294998)
 		(end 115.2 68.294998)
@@
 	)
 	(segment
+		(start 94.21 106.81)
+		(end 96.4 109)
+		(width 2)
+		(layer "B.Cu")
+		(net 1)
+	)
+	(segment
 		(start 150.971001 85.748999)
 		(end 152.34 84.38)
@@
 	)
 	(segment
+		(start 96.4 109)
+		(end 103.6 109)
+		(width 2)
+		(layer "B.Cu")
+		(net 1)
+	)
+	(segment
 		(start 120.2 68.294998)
 		(end 117.7 68.294998)
@@
 	)
 	(segment
+		(start 136.726041 106.726041)
+		(end 135.7 105.7)
+		(width 2)
+		(layer "B.Cu")
+		(net 1)
+	)
+	(segment
 		(start 112.883749 95.896041)
 		(end 110.45979 98.32)
@@
 	)
 	(segment
+		(start 143.75 106.726041)
+		(end 136.726041 106.726041)
+		(width 2)
+		(layer "B.Cu")
+		(net 1)
+	)
+	(segment
 		(start 122.75 67.45)
 		(end 121.044998 67.45)
@@
 	)
 	(segment
+		(start 104.4 108.2)
+		(end 110.371 102.229)
+		(width 2)
+		(layer "B.Cu")
+		(net 1)
+	)
+	(segment
 		(start 94.2 83.899999)
 		(end 94.2 82.71792)
@@
 	)
 	(segment
+		(start 104.4 108.2)
+		(end 104.4 104.37979)
+		(width 2)
+		(layer "B.Cu")
+		(net 1)
+	)
+	(segment
 		(start 94.2 70.322081)
 		(end 94.797919 70.92)
@@
 		(start 96.74 102.72)
 		(end 96.74 61.5)
-		(width 1.5)
+		(width 2)
 		(layer "F.Cu")
 		(net 2)
@@
 		(start 174.699 61.499)
 		(end 174.699 102.719)
-		(width 1.5)
+		(width 2)
 		(layer "F.Cu")
 		(net 2)
@@
 	)
 	(segment
+		(start 154.499 98.35)
+		(end 154.499 106.681)
+		(width 0.2)
+		(layer "F.Cu")
+		(net 35)
+	)
+	(segment
 		(start 114 84.7375)
 		(end 114.025 84.7625)
@@
 	)
 	(segment
-		(start 154.499 99.8)
-		(end 154.499 106.681)
-		(width 0.2)
-		(layer "F.Cu")
-		(net 35)
-	)
-	(segment
 		(start 114 80.6)
 		(end 114 84.7375)
@@
 	)
 	(via
-		(at 154.499 99.8)
+		(at 154.499 98.35)
 		(size 0.6)
 		(drill 0.3)
@@
 	)
 	(segment
+		(start 154.499 84.4)
+		(end 154.499 98.35)
+		(width 0.2)
+		(layer "B.Cu")
+		(net 35)
+	)
+	(segment
 		(start 116.6 77)
 		(end 123.101612 77)
@@
 	)
 	(segment
-		(start 154.499 84.4)
-		(end 154.499 99.8)
-		(width 0.2)
-		(layer "B.Cu")
-		(net 35)
-	)
-	(segment
 		(start 145.3 99.5671)
 		(end 149.849 104.1161)
@@
 	)
 	(segment
+		(start 153.898 97.65)
+		(end 153.899 97.651)
+		(width 0.2)
+		(layer "F.Cu")
+		(net 37)
+	)
+	(segment
 		(start 156.774 76.926)
 		(end 157.6 76.1)
@@
 	)
 	(segment
-		(start 152.16 106.84)
-		(end 151.8 106.84)
+		(start 153.899 97.651)
+		(end 153.899 105.101)
 		(width 0.2)
 		(layer "F.Cu")
@@
 	)
 	(segment
+		(start 152.16 106.84)
+		(end 151.8 106.84)
+		(width 0.2)
+		(layer "F.Cu")
+		(net 37)
+	)
+	(segment
 		(start 123.179 110.299)
 		(end 148.341 110.299)
@@
 	)
 	(segment
-		(start 153.899 101)
-		(end 153.899 105.101)
-		(width 0.2)
-		(layer "F.Cu")
-		(net 37)
-	)
-	(segment
 		(start 156.774 79.274)
 		(end 156.774 81.275057)
@@
 	)
 	(via
-		(at 153.899 101)
+		(at 153.898 97.65)
 		(size 0.6)
 		(drill 0.3)
@@
 	)
 	(segment
-		(start 153.899 85.3)
-		(end 153.898 85.301)
-		(width 0.2)
-		(layer "B.Cu")
-		(net 37)
-	)
-	(segment
 		(start 157.6 76.1)
 		(end 157.6 75.5)
@@
 	(segment
 		(start 153.898 85.301)
-		(end 153.898 100.999)
+		(end 153.899 85.3)
 		(width 0.2)
 		(layer "B.Cu")
@@
 	)
 	(segment
+		(start 153.898 97.65)
+		(end 153.898 85.301)
+		(width 0.2)
+		(layer "B.Cu")
+		(net 37)
+	)
+	(segment
 		(start 145.75 93.05)
 		(end 137.758223 85.058223)
@@
 	)
 	(segment
-		(start 153.898 100.999)
-		(end 153.899 101)
-		(width 0.2)
-		(layer "B.Cu")
-		(net 37)
-	)
-	(segment
 		(start 115.309768 78.940232)
 		(end 115.309768 79.2)
@@
 		(polygon
 			(pts
-				(xy 184.6 54.5) (xy 185.5 116.25) (xy 80.35 116.85) (xy 82.7 47.55)
+				(xy 179.05 113) (xy 179.05 59.7) (xy 161.3 59.7) (xy 158 56.4) (xy 113.2 56.4) (xy 109.9 59.7) (xy 92.4 59.75)
+				(xy 92.4 113)
 			)
 		)

Commit message: silk
Parts:
- added G***: LOGO, LOGO, F.Cu at (136.0, 67.0)
- added kibuzzard-690E9406: G***, kibuzzard-690E9406, F.Cu at (141.7, 73.8)
- added kibuzzard-690E9406: G***, kibuzzard-690E9406, F.Cu at (167.9, 90.8)
- added kibuzzard-690E9406: G***, kibuzzard-690E9406, F.Cu at (160.0, 94.2)
- added kibuzzard-690E9406: G***, kibuzzard-690E9406, F.Cu at (103.5, 94.2)
- added kibuzzard-690E9406: G***, kibuzzard-690E9406, F.Cu at (103.5, 79.5)
- added kibuzzard-690E9406: G***, kibuzzard-690E9406, F.Cu at (128.3, 86.4)
- added kibuzzard-690E9406: G***, kibuzzard-690E9406, F.Cu at (103.5, 61.1)
- added kibuzzard-690E9406: G***, kibuzzard-690E9406, F.Cu at (143.0, 92.5)
- added kibuzzard-690E9406: G***, kibuzzard-690E9406, F.Cu at (103.5, 101.8)
- added kibuzzard-690E9406: G***, kibuzzard-690E9406, F.Cu at (143.0, 81.2)
- added kibuzzard-690E9406: G***, kibuzzard-690E9406, F.Cu at (103.5, 74.5)
- added kibuzzard-690E9406: G***, kibuzzard-690E9406, F.Cu at (128.3, 92.6)
- added kibuzzard-690E9406: G***, kibuzzard-690E9406, F.Cu at (128.3, 90.1)
- added kibuzzard-690E9406: G***, kibuzzard-690E9406, F.Cu at (143.0, 83.8)
- added kibuzzard-690E9406: G***, kibuzzard-690E9406, F.Cu at (167.9, 79.7)
- added kibuzzard-690E9406: G***, kibuzzard-690E9406, F.Cu at (103.5, 66.1)
- added kibuzzard-690E9406: G***, kibuzzard-690E9406, F.Cu at (167.9, 74.7)
- added kibuzzard-690E9406: G***, kibuzzard-690E9406, F.Cu at (167.9, 102.0)
- added kibuzzard-690E9406: G***, kibuzzard-690E9406, F.Cu at (128.3, 83.9)
- added kibuzzard-690E9406: G***, kibuzzard-690E9406, F.Cu at (167.9, 68.5)
- added kibuzzard-690E9406: G***, kibuzzard-690E9406, F.Cu at (143.0, 95.0)
- added kibuzzard-690E9406: G***, kibuzzard-690E9406, F.Cu at (111.5, 74.0)
- added kibuzzard-690E9406: G***, kibuzzard-690E9406, F.Cu at (110.3, 65.7)
- added kibuzzard-690E9406: G***, kibuzzard-690E9406, F.Cu at (167.9, 94.5)
- added kibuzzard-690E9406: G***, kibuzzard-690E9406, F.Cu at (143.0, 78.8)
- added kibuzzard-690E9406: G***, kibuzzard-690E9406, F.Cu at (161.1, 97.5)
- added kibuzzard-690E9406: G***, kibuzzard-690E9406, F.Cu at (103.5, 99.2)
- added kibuzzard-690E9406: G***, kibuzzard-690E9406, F.Cu at (129.9, 68.8)
- added kibuzzard-690E9406: G***, kibuzzard-690E9406, F.Cu at (128.3, 78.9)
- added kibuzzard-690E9406: G***, kibuzzard-690E9406, F.Cu at (167.9, 63.5)
- added kibuzzard-690E9406: G***, kibuzzard-690E9406, F.Cu at (128.3, 97.6)
- added kibuzzard-690E9406: G***, kibuzzard-690E9406, F.Cu at (129.9, 73.8)
- added kibuzzard-690E9406: G***, kibuzzard-690E9406, F.Cu at (143.0, 90.0)
- added kibuzzard-690E9406: G***, kibuzzard-690E9406, F.Cu at (141.7, 71.3)
- added kibuzzard-690E9406: G***, kibuzzard-690E9406, F.Cu at (103.5, 83.3)
- added kibuzzard-690E9406: G***, kibuzzard-690E9406, F.Cu at (161.1, 102.5)
- added kibuzzard-690E9406: G***, kibuzzard-690E9406, F.Cu at (167.9, 77.2)
- added kibuzzard-690E9406: G***, kibuzzard-690E9406, F.Cu at (103.5, 77.0)
- added kibuzzard-690E9406: G***, kibuzzard-690E9406, F.Cu at (128.3, 95.1)
- added kibuzzard-690E9406: G***, kibuzzard-690E9406, F.Cu at (129.9, 71.3)
- added kibuzzard-690E9406: G***, kibuzzard-690E9406, F.Cu at (167.9, 66.0)
- added kibuzzard-690E9406: G***, kibuzzard-690E9406, F.Cu at (128.3, 81.4)
- added kibuzzard-690E9406: G***, kibuzzard-690E9406, F.Cu at (167.9, 72.2)
- added kibuzzard-690E9406: G***, kibuzzard-690E9406, F.Cu at (160.0, 91.7)
- added kibuzzard-690E9406: G***, kibuzzard-690E9406, F.Cu at (167.9, 99.5)
- added kibuzzard-690E9406: G***, kibuzzard-690E9406, F.Cu at (143.0, 86.2)
- added kibuzzard-690E9406: G***, kibuzzard-690E9406, F.Cu at (103.5, 96.8)
- added kibuzzard-690E9406: G***, kibuzzard-690E9406, F.Cu at (141.7, 68.8)
- added kibuzzard-690E9406: G***, kibuzzard-690E9406, F.Cu at (111.5, 69.0)
- added kibuzzard-690E9406: G***, kibuzzard-690E9406, F.Cu at (167.9, 61.0)
- added kibuzzard-690E9406: G***, kibuzzard-690E9406, F.Cu at (167.9, 85.8)
- added kibuzzard-690E9406: G***, kibuzzard-690E9406, F.Cu at (110.3, 63.2)
- added kibuzzard-690E9406: G***, kibuzzard-690E9406, F.Cu at (110.3, 60.7)
- added kibuzzard-690E9406: G***, kibuzzard-690E9406, F.Cu at (161.1, 100.0)
- added kibuzzard-690E9406: G***, kibuzzard-690E9406, F.Cu at (111.5, 71.5)
- added kibuzzard-690E9406: G***, kibuzzard-690E9406, F.Cu at (103.5, 88.3)
- added kibuzzard-690E9406: G***, kibuzzard-690E9406, F.Cu at (103.5, 63.6)
- added kibuzzard-690E9406: G***, kibuzzard-690E9406, F.Cu at (143.0, 97.5)
- added kibuzzard-690E9406: G***, kibuzzard-690E9406, F.Cu at (167.9, 88.3)
- added kibuzzard-690E9406: G***, kibuzzard-690E9406, F.Cu at (160.0, 89.2)
- added kibuzzard-690E9406: G***, kibuzzard-690E9406, F.Cu at (103.5, 90.8)
- added kibuzzard-690E9406: G***, kibuzzard-690E9406, F.Cu at (167.9, 83.3)
- added kibuzzard-690E9406: G***, kibuzzard-690E9406, F.Cu at (103.5, 85.8)
- added kibuzzard-690E9406: G***, kibuzzard-690E9406, B.Cu at (154.2, 62.5)
- added kibuzzard-690E9406: G***, kibuzzard-690E9406, B.Cu at (151.7, 62.5)
- added kibuzzard-690E9406: G***, kibuzzard-690E9406, B.Cu at (149.2, 62.5)
- added kibuzzard-690E9406: G***, kibuzzard-690E9406, F.Cu at (103.5, 68.6)
- added kibuzzard-690E9406: G***, kibuzzard-690E9406, B.Cu at (145.5, 62.5)
- added kibuzzard-690E9406: G***, kibuzzard-690E9406, B.Cu at (143.1, 69.8)
- added kibuzzard-690E9406: G***, kibuzzard-690E9406, B.Cu at (131.8, 62.5)
- added kibuzzard-690E9406: G***, kibuzzard-690E9406, B.Cu at (126.8, 62.5)
- added kibuzzard-690E9406: G***, kibuzzard-690E9406, B.Cu at (118.1, 62.5)
- added kibuzzard-690E9406: G***, kibuzzard-690E9406, B.Cu at (140.5, 62.5)
- added kibuzzard-690E9406: G***, kibuzzard-690E9406, B.Cu at (123.1, 62.5)
- added kibuzzard-690E9406: G***, kibuzzard-690E9406, B.Cu at (129.3, 62.5)
- added kibuzzard-690E9406: G***, kibuzzard-690E9406, B.Cu at (115.7, 69.8)
- added kibuzzard-690E9406: G***, kibuzzard-690E9406, B.Cu at (115.6, 62.5)
- added kibuzzard-690E9406: G***, kibuzzard-690E9406, F.Cu at (167.9, 97.0)
- added kibuzzard-690E9406: G***, kibuzzard-690E9406, B.Cu at (120.6, 62.5)
- added kibuzzard-690E9406: G***, kibuzzard-690E9406, B.Cu at (134.3, 62.5)
- added kibuzzard-690E9406: G***, kibuzzard-690E9406, B.Cu at (156.7, 62.5)
- added kibuzzard-690E9406: G***, kibuzzard-690E9406, B.Cu at (118.2, 69.8)
- added kibuzzard-690E9406: G***, kibuzzard-690E9406, B.Cu at (140.6, 69.8)
- added kibuzzard-690E9406: G***, kibuzzard-690E9406, B.Cu at (143.0, 62.5)
- added kibuzzard-690E9406: G***, kibuzzard-690E9406, B.Cu at (138.1, 69.8)
- added kibuzzard-690E9406: G***, kibuzzard-690E9406, B.Cu at (138.0, 62.5)
- added kibuzzard-690E9406: G***, kibuzzard-690E9406, B.Cu at (120.7, 69.8)
- added kibuzzard-690E9406: G***, kibuzzard-690E9406, F.Cu at (103.5, 72.0)
- added kibuzzard-690E943A: G***, kibuzzard-690E943A, F.Cu at (141.7, 69.8)
- added kibuzzard-690E943A: G***, kibuzzard-690E943A, F.Cu at (103.5, 97.8)
- added kibuzzard-690E943A: G***, kibuzzard-690E943A, F.Cu at (128.3, 96.2)
- added kibuzzard-690E943A: G***, kibuzzard-690E943A, F.Cu at (103.5, 95.3)
- added kibuzzard-690E943A: G***, kibuzzard-690E943A, F.Cu at (129.9, 69.9)
- added kibuzzard-690E943A: G***, kibuzzard-690E943A, F.Cu at (161.1, 98.5)
- added kibuzzard-690E943A: G***, kibuzzard-690E943A, F.Cu at (110.3, 64.2)
- added kibuzzard-690E943A: G***, kibuzzard-690E943A, F.Cu at (128.3, 98.7)
- added kibuzzard-690E943A: G***, kibuzzard-690E943A, F.Cu at (167.9, 86.9)
- added kibuzzard-690E943A: G***, kibuzzard-690E943A, F.Cu at (167.9, 78.2)
- added kibuzzard-690E943A: G***, kibuzzard-690E943A, F.Cu at (128.3, 82.5)
- added kibuzzard-690E943A: G***, kibuzzard-690E943A, F.Cu at (143.0, 93.5)
- added kibuzzard-690E943A: G***, kibuzzard-690E943A, F.Cu at (103.5, 62.1)
- added kibuzzard-690E943A: G***, kibuzzard-690E943A, F.Cu at (143.0, 91.0)
- added kibuzzard-690E943A: G***, kibuzzard-690E943A, F.Cu at (103.5, 91.8)
- added kibuzzard-690E943A: G***, kibuzzard-690E943A, F.Cu at (103.5, 80.6)
- added kibuzzard-690E943A: G***, kibuzzard-690E943A, F.Cu at (167.9, 84.4)
- added kibuzzard-690E943A: G***, kibuzzard-690E943A, F.Cu at (143.0, 82.3)
- added kibuzzard-690E943A: G***, kibuzzard-690E943A, F.Cu at (143.0, 98.5)
- added kibuzzard-690E943A: G***, kibuzzard-690E943A, F.Cu at (161.1, 103.5)
- added kibuzzard-690E943A: G***, kibuzzard-690E943A, F.Cu at (141.7, 74.8)
- added kibuzzard-690E943A: G***, kibuzzard-690E943A, F.Cu at (129.9, 74.9)
- added kibuzzard-690E943A: G***, kibuzzard-690E943A, F.Cu at (141.7, 72.3)
- added kibuzzard-690E943A: G***, kibuzzard-690E943A, F.Cu at (167.9, 69.6)
- added kibuzzard-690E943A: G***, kibuzzard-690E943A, F.Cu at (110.3, 66.7)
- added kibuzzard-690E943A: G***, kibuzzard-690E943A, F.Cu at (143.0, 84.8)
- added kibuzzard-690E943A: G***, kibuzzard-690E943A, F.Cu at (128.3, 91.2)
- added kibuzzard-690E943A: G***, kibuzzard-690E943A, F.Cu at (103.5, 78.1)
- added kibuzzard-690E943A: G***, kibuzzard-690E943A, F.Cu at (143.0, 96.0)
- added kibuzzard-690E943A: G***, kibuzzard-690E943A, F.Cu at (111.5, 75.0)
- added kibuzzard-690E943A: G***, kibuzzard-690E943A, F.Cu at (103.5, 64.6)
- added kibuzzard-690E943A: G***, kibuzzard-690E943A, F.Cu at (128.3, 80.0)
- added kibuzzard-690E943A: G***, kibuzzard-690E943A, F.Cu at (128.3, 87.5)
- added kibuzzard-690E943A: G***, kibuzzard-690E943A, F.Cu at (167.9, 100.6)
- added kibuzzard-690E943A: G***, kibuzzard-690E943A, F.Cu at (160.0, 92.8)
- added kibuzzard-690E943A: G***, kibuzzard-690E943A, F.Cu at (167.9, 95.6)
- added kibuzzard-690E943A: G***, kibuzzard-690E943A, F.Cu at (103.5, 75.6)
- added kibuzzard-690E943A: G***, kibuzzard-690E943A, F.Cu at (167.9, 89.4)
- added kibuzzard-690E943A: G***, kibuzzard-690E943A, F.Cu at (161.1, 101.0)
- added kibuzzard-690E943A: G***, kibuzzard-690E943A, F.Cu at (111.5, 72.5)
- added kibuzzard-690E943A: G***, kibuzzard-690E943A, F.Cu at (167.9, 98.1)
- added kibuzzard-690E943A: G***, kibuzzard-690E943A, F.Cu at (167.9, 73.2)
- added kibuzzard-690E943A: G***, kibuzzard-690E943A, F.Cu at (167.9, 67.1)
- added kibuzzard-690E943A: G***, kibuzzard-690E943A, F.Cu at (103.5, 102.8)
- added kibuzzard-690E943A: G***, kibuzzard-690E943A, F.Cu at (103.5, 73.1)
- added kibuzzard-690E943A: G***, kibuzzard-690E943A, F.Cu at (167.9, 103.1)
- added kibuzzard-690E943A: G***, kibuzzard-690E943A, F.Cu at (103.5, 67.1)
- added kibuzzard-690E943A: G***, kibuzzard-690E943A, F.Cu at (167.9, 75.7)
- added kibuzzard-690E943A: G***, kibuzzard-690E943A, F.Cu at (103.5, 86.8)
- added kibuzzard-690E943A: G***, kibuzzard-690E943A, F.Cu at (128.3, 93.7)
- added kibuzzard-690E943A: G***, kibuzzard-690E943A, F.Cu at (167.9, 64.6)
- added kibuzzard-690E943A: G***, kibuzzard-690E943A, F.Cu at (160.0, 90.3)
- added kibuzzard-690E943A: G***, kibuzzard-690E943A, F.Cu at (129.9, 72.4)
- added kibuzzard-690E943A: G***, kibuzzard-690E943A, F.Cu at (128.3, 85.0)
- added kibuzzard-690E943A: G***, kibuzzard-690E943A, F.Cu at (167.9, 91.9)
- added kibuzzard-690E943A: G***, kibuzzard-690E943A, F.Cu at (167.9, 62.1)
- added kibuzzard-690E943A: G***, kibuzzard-690E943A, F.Cu at (111.5, 70.0)
- added kibuzzard-690E943A: G***, kibuzzard-690E943A, F.Cu at (103.5, 84.3)
- added kibuzzard-690E943A: G***, kibuzzard-690E943A, F.Cu at (103.5, 100.3)
- added kibuzzard-690E943A: G***, kibuzzard-690E943A, F.Cu at (110.3, 61.7)
- added kibuzzard-690E943A: G***, kibuzzard-690E943A, F.Cu at (167.9, 80.7)
- added kibuzzard-690E943A: G***, kibuzzard-690E943A, F.Cu at (143.0, 79.8)
- added kibuzzard-690E943A: G***, kibuzzard-690E943A, F.Cu at (143.0, 87.3)
- added kibuzzard-690E943A: G***, kibuzzard-690E943A, B.Cu at (153.2, 62.5)
- added kibuzzard-690E943A: G***, kibuzzard-690E943A, B.Cu at (139.6, 69.8)
- added kibuzzard-690E943A: G***, kibuzzard-690E943A, B.Cu at (117.1, 62.5)
- added kibuzzard-690E943A: G***, kibuzzard-690E943A, F.Cu at (103.5, 89.3)
- added kibuzzard-690E943A: G***, kibuzzard-690E943A, B.Cu at (137.0, 62.5)
- added kibuzzard-690E943A: G***, kibuzzard-690E943A, B.Cu at (117.2, 69.8)
- added kibuzzard-690E943A: G***, kibuzzard-690E943A, B.Cu at (119.7, 69.8)
- added kibuzzard-690E943A: G***, kibuzzard-690E943A, B.Cu at (122.1, 62.5)
- added kibuzzard-690E943A: G***, kibuzzard-690E943A, B.Cu at (139.5, 62.5)
- added kibuzzard-690E943A: G***, kibuzzard-690E943A, B.Cu at (144.5, 62.5)
- added kibuzzard-690E943A: G***, kibuzzard-690E943A, B.Cu at (150.7, 62.5)
- added kibuzzard-690E943A: G***, kibuzzard-690E943A, B.Cu at (137.1, 69.8)
- added kibuzzard-690E943A: G***, kibuzzard-690E943A, B.Cu at (114.7, 69.8)
- added kibuzzard-690E943A: G***, kibuzzard-690E943A, B.Cu at (125.8, 62.5)
- added kibuzzard-690E943A: G***, kibuzzard-690E943A, F.Cu at (160.0, 95.3)
- added kibuzzard-690E943A: G***, kibuzzard-690E943A, B.Cu at (128.3, 62.5)
- added kibuzzard-690E943A: G***, kibuzzard-690E943A, B.Cu at (130.8, 62.5)
- added kibuzzard-690E943A: G***, kibuzzard-690E943A, B.Cu at (142.0, 62.5)
- added kibuzzard-690E943A: G***, kibuzzard-690E943A, B.Cu at (142.1, 69.8)
- added kibuzzard-690E943A: G***, kibuzzard-690E943A, B.Cu at (133.3, 62.5)
- added kibuzzard-690E943A: G***, kibuzzard-690E943A, B.Cu at (119.6, 62.5)
- added kibuzzard-690E943A: G***, kibuzzard-690E943A, B.Cu at (155.7, 62.5)
- added kibuzzard-690E943A: G***, kibuzzard-690E943A, B.Cu at (114.6, 62.5)
- added kibuzzard-690E943A: G***, kibuzzard-690E943A, B.Cu at (148.2, 62.5)
- added kibuzzard-690E943A: G***, kibuzzard-690E943A, F.Cu at (103.5, 69.6)
- added kibuzzard-6919B3C0: G***, kibuzzard-6919B3C0, F.Cu at (164.9, 82.1)
- added kibuzzard-6919B3C0: G***, kibuzzard-6919B3C0, F.Cu at (135.7, 93.3)
- added kibuzzard-6919B3C0: G***, kibuzzard-6919B3C0, F.Cu at (106.5, 81.9)
- added kibuzzard-6919B435: G***, kibuzzard-6919B435, B.Cu at (128.9, 67.0)
- added kibuzzard-6919B435: G***, kibuzzard-6919B435, B.Cu at (151.3, 67.0)
- added kibuzzard-6919B48D: G***, kibuzzard-6919B48D, F.Cu at (155.2, 105.6)
- added kibuzzard-6919B48D: G***, kibuzzard-6919B48D, F.Cu at (123.1, 105.6)
- C3: moved to B.Cu
- moved J2 0.40 mm to (104.5, 108.6)
Connections:
- H2 pad 1: unconnected-(H2-Pad1)_8 -> GND
Routing:
- net GND: track 573.6 -> 666.8 mm, vias 5 -> 6
- net +5VP: track 151.5 -> 219.3 mm
- net +5VPP: track 72.8 -> 118.6 mm
- net +3.3V: track 190.2 -> 191.6 mm
Other:
- board text added: "By Oscar Yosh GRIVELET"
- board text added: "Carte_extensions 2026_V1"
