File: carte ext/carte ext.kicad_sch (KiCad schematic)
At the start: 157 parts, among them J1 Conn_01x02, J10 Conn_01x04, J11 Conn_01x04, J12 Conn_01x04, J13 Conn_01x04, J14 Conn_01x04, J15 Conn_01x04, J16 Conn_01x04, J17 Conn_01x04, J18 Conn_01x04, J19 Conn_01x04, J2 Conn_01x02, J20 Conn_01x04, J21 Conn_02x04_Odd_Even, J22 Conn_02x04_Odd_Even, J23 Conn_02x04_Odd_Even, J24 Conn_02x04_Odd_Even, J25 Conn_02x04_Odd_Even, J26 Conn_02x04_Odd_Even, J27 Conn_02x04_Odd_Even, J28 Conn_02x04_Odd_Even, J29 Conn_02x04_Odd_Even, J3 Conn_01x04, J30 Conn_02x04_Odd_Even, J31 Conn_02x04_Odd_Even, J32 Conn_02x04_Odd_Even, J33 Conn_01x02, J4 Conn_01x04, J5 Conn_01x04, J6 Conn_01x04, J7 Conn_01x04, J8 Conn_01x04, J9 Conn_01x04, U1 PCA9685PW, U2 PCA9685PW, U3 PCA9685PW, U4 PCF8574AT, U5 PCF8574AT

Commit message: silk
Connections:
- net GND: now also H2.1
- no-connect marks 1 -> 0
Changed lines of the file:
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@@
 		(color 0 0 0 0)
 	)
-	(no_connect
-		(at 49.53 251.46)
-	)
 	(wire
 		(pts
@@
 					(unit 1)
 				)
+			)
+		)
+	)
+	(symbol
+		(lib_name "GND_2")
+		(lib_id "power:GND")
+		(at 49.53 251.46 0)
+		(unit 1)
+		(exclude_from_sim no)
+		(in_bom yes)
+		(on_board yes)
+		(dnp no)
+		(fields_autoplaced yes)
+		(property "Reference" "#PWR010"
+			(at 49.53 257.81 0)
+			(effects
+				(font
+					(size 1.27 1.27)
+				)
+				(hide yes)
+			)
+		)
+		(property "Value" "GND"
+			(at 49.53 256.54 0)
+			(effects
+				(font
+					(size 1.27 1.27)
+				)
+			)
+		)
+		(property "Footprint" ""
+			(at 49.53 251.46 0)
+			(effects
+				(font
+					(size 1.27 1.27)
+				)
+				(hide yes)
+			)
+		)
+		(property "Datasheet" ""
+			(at 49.53 251.46 0)
+			(effects
+				(font
+					(size 1.27 1.27)
+				)
+				(hide yes)
+			)
+		)
+		(property "Description" "Power symbol creates a global label with name \"GND\" , ground"
+			(at 49.53 251.46 0)
+			(effects
+				(font
+					(size 1.27 1.27)
+				)
+				(hide yes)
+			)
+		)
+		(pin "1"
+		)
+		(instances
+			(project "carte ext"
+				(path "/560e5d6e-957e-4a7b-943a-ee18f8c29f91"
+					(reference "#PWR010")
+					(unit 1)
+				)

Commit message: xt30
Parts:
- J1, J2, J33: footprint Connector_AMASS:AMASS_XT60-F_1x02_P7.20mm_Vertical -> Connector_AMASS:AMASS_XT30U-F_1x02_P5.0mm_Vertical
Changed lines of the file:
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@@
 			)
 		)
-		(property "Footprint" "Connector_AMASS:AMASS_XT60-F_1x02_P7.20mm_Vertical"
+		(property "Footprint" "Connector_AMASS:AMASS_XT30U-F_1x02_P5.0mm_Vertical"
 			(at 311.15 34.29 0)
 			(effects
@@
 			)
 		)
-		(property "Footprint" "Connector_AMASS:AMASS_XT60-F_1x02_P7.20mm_Vertical"
+		(property "Footprint" "Connector_AMASS:AMASS_XT30U-F_1x02_P5.0mm_Vertical"
 			(at 311.15 41.91 0)
 			(effects
@@
 			)
 		)
-		(property "Footprint" "Connector_AMASS:AMASS_XT60-F_1x02_P7.20mm_Vertical"
+		(property "Footprint" "Connector_AMASS:AMASS_XT30U-F_1x02_P5.0mm_Vertical"
 			(at 311.15 26.67 0)
 			(effects
